File: PineWoodDerby-Mega_Shield.brd (EAGLE design)
At the start: 101.6 x 53.3 mm, 43 parts, among them CN1 RJ45-8PTH, CN2 RJ45-8PTH, CN3 RJ45-8PTH, CN4 RJ45-8PTH, Q1 MOSFET-PCHANNELFQP27P06, Q2 MOSFET-PCHANNELFQP27P06, Q3 MOSFET-PCHANNELFQP27P06, U1 MAX232PTH, U2 MAX3232

Commit message: update
Parts:
- removed C10, C11, C7, C8, C9: 0.1uF, SparkFun-Capacitors:CAP-PTH-SMALL-KIT
- removed U$2: CREATIVE_COMMONS, SparkFun:CREATIVE_COMMONS
- removed U1: MAX232PTH, SparkFun-DigitalIC:DIL16
Connections:
- removed net N$10: C9.1, U1.2
- removed net N$3: C7.1, U1.1
- removed net N$4: C7.2, U1.3
- removed net N$6: C8.1, U1.4
- removed net N$7: C8.2, U1.5
- removed net N$8: C10.2, C11.2, C9.2
- removed net N$9: C10.1, U1.6
- net 5V: no longer C11.1, U1.16
Other:
- board size 101.6 x 53.3 mm -> 104.1 x 81.3 mm
Changed lines of the file:
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@@
 <wire x1="64.135" y1="46.99" x2="63.5" y2="46.99" width="0.4064" layer="21"/>
 <wire x1="63.5" y1="46.99" x2="63.5" y2="46.355" width="0.4064" layer="21"/>
-<wire x1="0" y1="0" x2="99.06" y2="0" width="0.254" layer="51"/>
-<wire x1="99.06" y1="0" x2="99.06" y2="1.27" width="0.254" layer="51"/>
-<wire x1="99.06" y1="1.27" x2="101.6" y2="3.81" width="0.254" layer="51"/>
-<wire x1="101.6" y1="3.81" x2="101.6" y2="38.1" width="0.254" layer="51"/>
-<wire x1="101.6" y1="38.1" x2="99.06" y2="40.64" width="0.254" layer="51"/>
-<wire x1="99.06" y1="40.64" x2="99.06" y2="50.8" width="0.254" layer="51"/>
-<wire x1="99.06" y1="50.8" x2="96.52" y2="53.34" width="0.254" layer="51"/>
-<wire x1="96.52" y1="53.34" x2="0" y2="53.34" width="0.254" layer="51"/>
-<wire x1="0" y1="53.34" x2="0" y2="0" width="0.254" layer="51"/>
+<wire x1="0" y1="0" x2="104.14" y2="0" width="0.254" layer="51"/>
+<wire x1="104.14" y1="0" x2="104.14" y2="81.28" width="0.254" layer="51"/>
+<wire x1="104.14" y1="81.28" x2="0" y2="81.28" width="0.254" layer="51"/>
+<wire x1="0" y1="81.28" x2="0" y2="0" width="0.254" layer="51"/>
 <wire x1="1.27" y1="39.37" x2="1.27" y2="36.83" width="0.2032" layer="21"/>
-<wire x1="0" y1="0" x2="99.06" y2="0" width="0.2032" layer="20"/>
-<wire x1="99.06" y1="0" x2="99.06" y2="1.27" width="0.2032" layer="20"/>
-<wire x1="99.06" y1="1.27" x2="101.6" y2="3.81" width="0.2032" layer="20"/>
-<wire x1="101.6" y1="3.81" x2="101.6" y2="38.1" width="0.2032" layer="20"/>
-<wire x1="101.6" y1="38.1" x2="99.06" y2="40.64" width="0.2032" layer="20"/>
-<wire x1="99.06" y1="40.64" x2="99.06" y2="50.8" width="0.2032" layer="20"/>
-<wire x1="99.06" y1="50.8" x2="96.52" y2="53.34" width="0.2032" layer="20"/>
-<wire x1="96.52" y1="53.34" x2="0" y2="53.34" width="0.2032" layer="20"/>
-<wire x1="0" y1="53.34" x2="0" y2="0" width="0.2032" layer="20"/>
+<wire x1="0" y1="0" x2="104.14" y2="0" width="0.2032" layer="20"/>
+<wire x1="104.14" y1="0" x2="104.14" y2="81.28" width="0.2032" layer="20"/>
+<wire x1="104.14" y1="81.28" x2="0" y2="81.28" width="0.2032" layer="20"/>
+<wire x1="0" y1="81.28" x2="0" y2="0" width="0.2032" layer="20"/>
 <text x="64.135" y="6.985" size="1.6764" layer="21" font="vector" ratio="15">ANALOG IN</text>
 <text x="24.4812" y="44.1828" size="1.4224" layer="21" font="vector" ratio="15" rot="R90">AREF</text>
@@
 <attribute name="VALUE" x="19.177" y="5.969" size="0.8128" layer="21" ratio="15" rot="R180"/>
 </element>
-<element name="U$2" library="SparkFun" package="CREATIVE_COMMONS" value="CREATIVE_COMMONS" x="20.32" y="-7.62"/>
 <element name="CN1" library="SparkFun-Connectors" package="RJ45-8" value="RJ45-8PTH" x="27.94" y="71.12" rot="MR180">
 <attribute name="LABEL" value="Start Sensors" x="27.94" y="71.12" size="1.778" layer="28" rot="MR180" display="off"/>
@@
 <element name="SJ2" library="SparkFun" package="SJ_2S-TRACE" value="SOLDERJUMPERTRACE" x="74.93" y="17.78" rot="R180"/>
 <element name="C6" library="SparkFun" package="0402-CAP" value="0.1uF" x="78.74" y="17.78" rot="R180"/>
-<element name="U1" library="SparkFun-DigitalIC" package="DIL16" value="MAX232PTH" x="10.16" y="20.32" rot="R270"/>
-<element name="C7" library="SparkFun-Capacitors" package="CAP-PTH-SMALL-KIT" value="0.1uF" x="2.54" y="26.67" rot="R270">
-<attribute name="PROD_ID" value="CAP-08370" x="2.54" y="26.67" size="1.778" layer="27" rot="R270" display="off"/>
-</element>
-<element name="C8" library="SparkFun-Capacitors" package="CAP-PTH-SMALL-KIT" value="0.1uF" x="2.54" y="19.05" rot="R270">
-<attribute name="PROD_ID" value="CAP-08370" x="2.54" y="19.05" size="1.778" layer="27" rot="R270" display="off"/>
-</element>
-<element name="C9" library="SparkFun-Capacitors" package="CAP-PTH-SMALL-KIT" value="0.1uF" x="10.16" y="25.4" rot="R270">
-<attribute name="PROD_ID" value="CAP-08370" x="10.16" y="25.4" size="1.778" layer="27" rot="R270" display="off"/>
-</element>
-<element name="C10" library="SparkFun-Capacitors" package="CAP-PTH-SMALL-KIT" value="0.1uF" x="10.16" y="19.05" rot="R90">
-<attribute name="PROD_ID" value="CAP-08370" x="10.16" y="19.05" size="1.778" layer="27" rot="R90" display="off"/>
-</element>
-<element name="C11" library="SparkFun-Capacitors" package="CAP-PTH-SMALL-KIT" value="0.1uF" x="11.43" y="25.4" rot="R270">
-<attribute name="PROD_ID" value="CAP-08370" x="11.43" y="25.4" size="1.778" layer="27" rot="R270" display="off"/>
-</element>
 </elements>
 <signals>
@@
 <contactref element="Q2" pad="2"/>
 <contactref element="Q1" pad="2"/>
-<contactref element="U1" pad="16"/>
-<contactref element="C11" pad="1"/>
 <wire x1="76.46" y1="29.845" x2="78.725" y2="29.845" width="0.4064" layer="1"/>
 <wire x1="78.725" y1="29.845" x2="78.74" y2="29.86" width="0.4064" layer="1"/>
 <wire x1="38.1" y1="2.54" x2="76.46" y2="29.845" width="0" layer="19" extent="1-1"/>
-<wire x1="11.43" y1="26.797" x2="21.717" y2="7.747" width="0" layer="19" extent="1-1"/>
-<wire x1="13.97" y1="29.21" x2="11.43" y2="26.797" width="0" layer="19" extent="1-1"/>
-<wire x1="17.78" y1="57.15" x2="13.97" y2="29.21" width="0" layer="19" extent="1-1"/>
+<wire x1="17.78" y1="57.15" x2="21.717" y2="7.747" width="0" layer="19" extent="1-1"/>
 <wire x1="34.29" y1="57.15" x2="17.78" y2="57.15" width="0" layer="19" extent="1-1"/>
 </signal>
@@
 <polygon width="0.2032" layer="16" isolate="0.3048">
 <vertex x="0" y="0"/>
-<vertex x="99.06" y="0"/>
-<vertex x="99.06" y="1.27"/>
-<vertex x="101.6" y="3.81"/>
-<vertex x="101.6" y="38.1"/>
-<vertex x="99.06" y="40.64"/>
-<vertex x="99.06" y="50.8"/>
-<vertex x="96.52" y="53.34"/>
-<vertex x="0" y="53.34"/>
+<vertex x="104.14" y="0"/>
+<vertex x="104.14" y="81.28"/>
+<vertex x="0" y="81.28"/>
 </polygon>
 <polygon width="0.2032" layer="1" isolate="0.3048">
 <vertex x="0" y="0"/>
-<vertex x="99.06" y="0"/>
-<vertex x="99.06" y="1.27"/>
-<vertex x="101.6" y="3.81"/>
-<vertex x="101.6" y="38.1"/>
-<vertex x="99.06" y="40.64"/>
-<vertex x="99.06" y="50.8"/>
-<vertex x="96.52" y="53.34"/>
-<vertex x="0" y="53.34"/>
+<vertex x="104.14" y="0"/>
+<vertex x="104.14" y="81.28"/>
+<vertex x="0" y="81.28"/>
 </polygon>
 <contactref element="U2" pad="15"/>
@@
 <wire x1="78.09" y1="17.78" x2="75.438" y2="17.78" width="0" layer="19" extent="1-1"/>
 </signal>
-<signal name="N$3">
-<contactref element="U1" pad="1"/>
-<contactref element="C7" pad="1"/>
-<wire x1="2.54" y1="28.067" x2="6.35" y2="29.21" width="0" layer="19" extent="1-1"/>
-</signal>
-<signal name="N$4">
-<contactref element="C7" pad="2"/>
-<contactref element="U1" pad="3"/>
-<wire x1="2.54" y1="25.273" x2="6.35" y2="24.13" width="0" layer="19" extent="1-1"/>
-</signal>
-<signal name="N$6">
-<contactref element="C8" pad="1"/>
-<contactref element="U1" pad="4"/>
-<wire x1="2.54" y1="20.447" x2="6.35" y2="21.59" width="0" layer="19" extent="1-1"/>
-</signal>
-<signal name="N$7">
-<contactref element="C8" pad="2"/>
-<contactref element="U1" pad="5"/>
-<wire x1="2.54" y1="17.653" x2="6.35" y2="19.05" width="0" layer="19" extent="1-1"/>
-</signal>
-<signal name="N$8">
-<contactref element="C11" pad="2"/>
-<contactref element="C10" pad="2"/>
-<contactref element="C9" pad="2"/>
-<wire x1="10.16" y1="24.003" x2="11.43" y2="24.003" width="0" layer="19" extent="1-1"/>
-<wire x1="10.16" y1="20.447" x2="10.16" y2="24.003" width="0" layer="19" extent="1-1"/>
-</signal>
-<signal name="N$9">
-<contactref element="C10" pad="1"/>
-<contactref element="U1" pad="6"/>
-<wire x1="6.35" y1="16.51" x2="10.16" y2="17.653" width="0" layer="19" extent="1-1"/>
-</signal>
-<signal name="N$10">
-<contactref element="U1" pad="2"/>
-<contactref element="C9" pad="1"/>
-<wire x1="6.35" y1="26.67" x2="10.16" y2="26.797" width="0" layer="19" extent="1-1"/>
-</signal>
 <signal name="N$11">
