File: PineWoodDerby-Mega_Shield.sch (EAGLE design)
At the start: 43 parts, among them CN1 RJ45-8PTH, CN2 RJ45-8PTH, CN3 RJ45-8PTH, CN4 RJ45-8PTH, Q1 MOSFET-PCHANNELFQP27P06, Q2 MOSFET-PCHANNELFQP27P06, Q3 MOSFET-PCHANNELFQP27P06, U1 MAX232PTH, U2 MAX3232

Commit message: update
Parts:
- removed C10, C11, C7, C8, C9: 0.1uF, SparkFun-Capacitors:0.1UF-50V-20%(PTH)KIT-EZ
- removed U$2: CREATIVE_COMMONS, SparkFun:CREATIVE_COMMONS
- removed U1: MAX232PTH, SparkFun-DigitalIC:MAX232PTH
Connections:
- removed net N$10: C9.1, U1.V+
- removed net N$3: C7.1, U1.C1+
- removed net N$4: C7.2, U1.C1-
- removed net N$6: C8.1, U1.C2+
- removed net N$7: C8.2, U1.C2-
- removed net N$8: C10.2, C11.2, C9.2
- removed net N$9: C10.1, U1.V-
- net 5V: no longer C11.1, U1.VCC
Other:
- note removed: "3.0V < VCC < 5.5V"
- note removed: "Ryan Owens"
- moved on the sheet: C1, C2, C3, C4, C5, C6, CN4, Q3, SJ2, U$1, U$3, U2
