File: PineWoodDerby_Mega_Shield.brd (EAGLE design)
At the start: 104.1 x 81.3 mm, 36 parts, among them CN1 RJ45-8PTH, CN2 RJ45-8PTH, CN3 RJ45-8PTH, CN4 RJ45-8PTH, Q1 MOSFET-PCHANNELFQP27P06, Q2 MOSFET-PCHANNELFQP27P06, Q3 MOSFET-PCHANNELFQP27P06, U2 MAX3232

Commit message: update
Parts:
- removed C6: 0.1uF, SparkFun:0402-CAP
- removed SJ2: SOLDERJUMPERTRACE, SparkFun:SJ_2S-TRACE
- moved R1 17.8 mm to (2.41, 14.0), turned to 90 degrees
- moved R2 14.5 mm to (5.08, 14.0), turned to 90 degrees
- moved R3 13.9 mm to (8.00, 14.0), turned to 90 degrees
- moved C2 10.2 mm to (68.6, 35.6)
- moved C4 10.2 mm to (67.3, 35.6)
- moved U2 10.2 mm to (73.7, 35.6)
- moved C1 10.2 mm to (68.6, 39.4)
- moved C3 10.2 mm to (67.3, 39.4)
- moved C5 10.2 mm to (78.7, 39.4)
- moved LED1 6.35 mm to (3.81, 5.08), turned to 270 degrees
- moved LED2 6.35 mm to (10.2, 5.08), turned to 270 degrees
- moved S1 5.34 mm to (22.6, 5.08), turned to 180 degrees
- moved Q3 2.54 mm to (63.5, 57.1)
Connections:
- removed net DIO3: SJ2.2, U$1.17
- removed net N$5: C6.2, SJ2.1
- net D22: now also U$1.20
- net D24: now also U$1.19
- net D26: now also U$1.16
- net D28: now also U$1.14
- net D30: now also U$1.12
- net D32: now also U$1.4
- net D34: now also U$1.5
- net D36: now also U$1.6
- net D38: now also U$1.7
- net D40: now also U$1.8
- net D42: now also U$1.9
- net RES: no longer C6.1
Routing:
- net VIN: track 0.00 -> 163.6 mm
- net 3.3: track 0.51 -> 100.7 mm
- net RES: track 122.5 -> 28.2 mm
- net 5V: track 28.3 -> 120.0 mm, vias 1 -> 3
- net D13: track 43.3 -> 0.00 mm
- net D30: track 0.00 -> 40.1 mm
- net D28: track 0.00 -> 38.7 mm
- net D26: track 0.00 -> 36.7 mm
- net D24: track 0.00 -> 35.6 mm
- net D22: track 0.00 -> 34.5 mm
- net ARM_LED: track 0.00 -> 23.7 mm
- net TRIGGER: track 0.00 -> 20.9 mm
- net TXD1: track 1.03 -> 21.7 mm
- net RXD1: track 1.03 -> 21.1 mm
- net GND: track 4.80 -> 23.9 mm
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