File: PineWoodDerby_Mega_Shield.sch (EAGLE design)
At the start: 36 parts, among them CN1 RJ45-8PTH, CN2 RJ45-8PTH, CN3 RJ45-8PTH, CN4 RJ45-8PTH, Q1 MOSFET-PCHANNELFQP27P06, Q2 MOSFET-PCHANNELFQP27P06, Q3 MOSFET-PCHANNELFQP27P06, U2 MAX3232

Commit message: update
Parts:
- removed C6: 0.1uF, SparkFun:CAP0402-CAP
- removed SJ2: SOLDERJUMPERTRACE, SparkFun:SOLDERJUMPERTRACE
Connections:
- removed net DIO3: SJ2.2, U$1.DIO3
- removed net N$5: C6.2, SJ2.1
- net D22: now also U$1.DIO0
- net D24: now also U$1.DIO1
- net D26: now also U$1.RTS
- net D28: now also U$1.RES@14
- net D30: now also U$1.CTS
- net D32: now also U$1.DIO12
- net D34: now also U$1.RESET
- net D36: now also U$1.RSSI
- net D38: now also U$1.DIO11
- net D40: now also U$1.RES@8
- net D42: now also U$1.DTR
- net RES: no longer C6.1
Changed lines of the file:
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@@
 <part name="U$1" library="SparkFun-RF" deviceset="XBEE-2" device="B2"/>
 <part name="GND10" library="SparkFun" deviceset="GND" device=""/>
-<part name="SJ2" library="SparkFun" deviceset="SOLDERJUMPER" device="TRACE"/>
-<part name="C6" library="SparkFun" deviceset="CAP" device="0402-CAP" value="0.1uF"/>
 <part name="P+5" library="SparkFun-Aesthetics" deviceset="VCC" device="" value="3.3"/>
 <part name="VIN" library="SparkFun-Aesthetics" deviceset="VCC" device="" value="VIN"/>
@@
 <instance part="U$1" gate="G$1" x="236.22" y="129.54"/>
 <instance part="GND10" gate="1" x="215.9" y="111.76"/>
-<instance part="SJ2" gate="1" x="269.24" y="132.08" rot="R180"/>
-<instance part="C6" gate="G$1" x="287.02" y="132.08" rot="R270"/>
 <instance part="P+5" gate="1" x="215.9" y="142.24"/>
 <instance part="VIN" gate="1" x="167.64" y="220.98" rot="MR0"/>
@@
 <pinref part="S1" gate="S" pin="4"/>
 <pinref part="S1" gate="S" pin="3"/>
-</segment>
-<segment>
-<wire x1="292.1" y1="132.08" x2="302.26" y2="132.08" width="0.1524" layer="91"/>
-<label x="302.26" y="132.08" size="1.778" layer="95" rot="R180"/>
-<pinref part="C6" gate="G$1" pin="1"/>
 </segment>
 </net>
@@
 <pinref part="JP9" gate="G$1" pin="1"/>
 </segment>
+<segment>
+<wire x1="256.54" y1="139.7" x2="264.16" y2="139.7" width="0.1524" layer="91"/>
+<pinref part="U$1" gate="G$1" pin="DIO0"/>
+<label x="264.16" y="139.7" size="1.778" layer="95"/>
+</segment>
 </net>
 <net name="D24" class="0">
@@
 <pinref part="JP9" gate="G$1" pin="2"/>
 </segment>
-</net>
-<net name="D26" class="0">
-<segment>
-<wire x1="170.18" y1="157.48" x2="172.72" y2="157.48" width="0.1524" layer="91"/>
-<label x="169.672" y="158.242" size="1.778" layer="95" rot="R180"/>
-<pinref part="JP9" gate="G$1" pin="3"/>
+<segment>
+<wire x1="256.54" y1="137.16" x2="264.16" y2="137.16" width="0.1524" layer="91"/>
+<label x="264.16" y="137.16" size="1.778" layer="95"/>
+<pinref part="U$1" gate="G$1" pin="DIO1"/>
 </segment>
 </net>
@@
 <pinref part="JP9" gate="G$1" pin="4"/>
 </segment>
+<segment>
+<label x="261.62" y="124.46" size="1.778" layer="95"/>
+<wire x1="256.54" y1="124.46" x2="261.62" y2="124.46" width="0.1524" layer="91"/>
+<pinref part="U$1" gate="G$1" pin="RES@14"/>
+</segment>
 </net>
 <net name="D30" class="0">
@@
 <pinref part="JP9" gate="G$1" pin="5"/>
 </segment>
+<segment>
+<label x="261.62" y="119.38" size="1.778" layer="95"/>
+<wire x1="256.54" y1="119.38" x2="261.62" y2="119.38" width="0.1524" layer="91"/>
+<pinref part="U$1" gate="G$1" pin="CTS"/>
+</segment>
 </net>
 <net name="D32" class="0">
@@
 <pinref part="JP9" gate="G$1" pin="6"/>
 </segment>
+<segment>
+<wire x1="213.36" y1="132.08" x2="215.9" y2="132.08" width="0.1524" layer="91"/>
+<label x="208.28" y="132.08" size="1.778" layer="95"/>
+<pinref part="U$1" gate="G$1" pin="DIO12"/>
+</segment>
 </net>
 <net name="D34" class="0">
@@
 <pinref part="JP9" gate="G$1" pin="7"/>
 </segment>
+<segment>
+<wire x1="213.36" y1="129.54" x2="215.9" y2="129.54" width="0.1524" layer="91"/>
+<pinref part="U$1" gate="G$1" pin="RESET"/>
+<label x="208.28" y="129.54" size="1.778" layer="95"/>
+</segment>
 </net>
 <net name="D36" class="0">
@@
 <pinref part="JP9" gate="G$1" pin="8"/>
 </segment>
+<segment>
+<wire x1="213.36" y1="127" x2="215.9" y2="127" width="0.1524" layer="91"/>
+<pinref part="U$1" gate="G$1" pin="RSSI"/>
+<label x="208.28" y="127" size="1.778" layer="95"/>
+</segment>
 </net>
 <net name="D38" class="0">
@@
 <pinref part="JP9" gate="G$1" pin="9"/>
 </segment>
+<segment>
+<wire x1="213.36" y1="124.46" x2="215.9" y2="124.46" width="0.1524" layer="91"/>
+<pinref part="U$1" gate="G$1" pin="DIO11"/>
+<label x="208.28" y="124.46" size="1.778" layer="95"/>
+</segment>
 </net>
 <net name="D40" class="0">
@@
 <pinref part="JP9" gate="G$1" pin="10"/>
 </segment>
+<segment>
+<wire x1="213.36" y1="121.92" x2="215.9" y2="121.92" width="0.1524" layer="91"/>
+<pinref part="U$1" gate="G$1" pin="RES@8"/>
+<label x="208.28" y="121.92" size="1.778" layer="95"/>
+</segment>
 </net>
 <net name="D42" class="0">
@@
 <label x="169.672" y="138.684" size="1.778" layer="95" rot="R180"/>
 <pinref part="JP9" gate="G$1" pin="11"/>
+</segment>
+<segment>
+<wire x1="213.36" y1="119.38" x2="215.9" y2="119.38" width="0.1524" layer="91"/>
+<label x="208.28" y="119.38" size="1.778" layer="95"/>
+<pinref part="U$1" gate="G$1" pin="DTR"/>
 </segment>
 </net>
@@
 </segment>
 </net>
-<net name="DIO3" class="0">
-<segment>
-<wire x1="264.16" y1="132.08" x2="256.54" y2="132.08" width="0.1524" layer="91"/>
-<label x="259.08" y="132.08" size="1.778" layer="95"/>
-<pinref part="SJ2" gate="1" pin="2"/>
-<pinref part="U$1" gate="G$1" pin="DIO3"/>
-</segment>
-</net>
-<net name="N$5" class="0">
-<segment>
-<wire x1="284.48" y1="132.08" x2="274.32" y2="132.08" width="0.1524" layer="91"/>
-<pinref part="SJ2" gate="1" pin="1"/>
-<pinref part="C6" gate="G$1" pin="2"/>
-</segment>
-</net>
 <net name="N$11" class="0">
 <segment>
@@
 </segment>
 </net>
+<net name="D26" class="0">
+<segment>
+<wire x1="170.18" y1="157.48" x2="172.72" y2="157.48" width="0.1524" layer="91"/>
+<label x="169.672" y="158.242" size="1.778" layer="95" rot="R180"/>
+<pinref part="JP9" gate="G$1" pin="3"/>
+</segment>
+<segment>
+<label x="261.62" y="129.54" size="1.778" layer="95"/>
+<wire x1="256.54" y1="129.54" x2="261.62" y2="129.54" width="0.1524" layer="91"/>
+<pinref part="U$1" gate="G$1" pin="RTS"/>
+</segment>
+</net>
